File: KiCad_ch32v203_F6P6/KiCad_ch32v203_F6P6.kicad_pcb (KiCad board)
At the start: 2 copper layers, 26 x 51 mm, 26 parts, among them J1 Header1, J2 Header2, J3 SWD, SW1 BT0, SW2 RST, U1 AMS1117-3.3, U2 CH32V203F6P6, Y1 8Mhz

Commit message: Rell!
Parts:
- moved J3 0.67 mm to (126.3, 68.0)
- moved USB1 0.20 mm to (130.0, 25.4)
Routing:
- net GND: track 207.1 -> 198.9 mm
- net /SWDIO: track 45.4 -> 46.1 mm
- net VBUS: track 23.5 -> 22.8 mm
- net /PA12: track 59.7 -> 60.3 mm
Other:
- board text added: "3V3"
- board text added: "3v3"
- board text added: "BT0"
- board text added: "CLK"
- board text added: "GND"
- board text added: "PA0"
- board text added: "PA1"
- board text added: "PA11"
- board text added: "PA12"
- board text added: "PA2"
- board text added: "PA4"
- board text added: "PA5"
- board text added: "PA6"
- board text added: "PA7"
- board text added: "PB1"
- board text added: "RST"
- board text added: "SIO"
- board text added: "SLK"
- board text added: "TAUNOE"
- board text added: "V1 2025"
- board text added: "VBUS"
- board text added: "X0"
- board text added: "XI"

Commit message: kicad silkscreen
Parts:
- moved J3 0.20 mm to (126.3, 67.8)
Routing:
- net GND: track 198.9 -> 200.7 mm
- net /PA11: track 60.8 -> 59.9 mm
- net /SWDIO: track 46.1 -> 45.3 mm
- net /Reset BTN: track 50.1 -> 50.6 mm
- added copper zone on B.Cu, net GND
Other:
- board text added: "DIO"
- board text added: "PA3"
- board text added: "SCLK"
- board text added: "SDIO"
- board text removed: "SLK"

Commit message: board ready
Parts:
- J1, J2: moved to B.Cu
- USB1: footprint Connector_USB:USB_C_Receptacle_Palconn_UTC16-G -> Connector_USB:USB_C_Receptacle_HCTL_HC-TYPE-C-16P-01A
- Y1: footprint Crystal:Crystal_SMD_5032-2Pin_5.0x3.2mm_HandSoldering -> Crystal:Crystal_SMD_5032-2Pin_5.0x3.2mm
- moved C2 55.3 mm to (141.7, 89.1)
- moved C5 55.3 mm to (157.2, 78.1)
- moved C7 55.3 mm to (143.2, 98.8)
- moved C8 55.3 mm to (149.9, 98.8)
- moved J2 55.3 mm to (155.3, 89.0), turned to 180 degrees
- moved J3 55.3 mm to (142.8, 120.6)
- moved LED2 55.3 mm to (145.1, 117.4)
- moved R2 55.3 mm to (157.2, 83.3)
- moved R3 55.3 mm to (135.8, 83.5)
- moved R4 55.3 mm to (154.2, 84.5)
- moved R6 55.3 mm to (150.2, 117.4)
- moved SW2 55.3 mm to (154.2, 78.8)
- moved C1 55.3 mm to (148.9, 84.2)
- moved C6 55.3 mm to (135.8, 78.2)
- moved F1 55.3 mm to (143.6, 84.2)
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Routing:
- net GND: track 200.7 -> 203.4 mm
- net /Reset BTN: track 50.6 -> 48.9 mm
- net +3.3V: track 99.0 -> 100.6 mm
- net /BOOT0 BTN: track 49.9 -> 48.6 mm
- net /SWDIO: track 45.3 -> 44.4 mm
- net /SWCLK: track 47.1 -> 46.2 mm
- net /OSC_OUT: track 35.2 -> 34.4 mm
- net /PA11: track 59.9 -> 59.1 mm
- net Net-(U1-VI): track 7.84 -> 7.26 mm
- net /OSC_IN: track 18.0 -> 17.5 mm
Other:
- board text added: "Designed in Estonia"
- board text added: "github.com/taunoe/ Taunoe_CH32V203"
