File: KiCad_ch32v203_F6P6/KiCad_ch32v203_F6P6.kicad_sch (KiCad schematic)
At the start: 26 parts, among them J1 SWD, J2 USB_C_Receptacle_USB2.0_16P, J3 Conn_01x12_Pin, J4 Conn_01x12_Pin, SW1 RST, SW2 BT0, U1 CH32V203F6P6, U2 AMS1117-3.3, Y1 8Mhz

Commit message: started board file
Parts:
- removed J3, J4: Conn_01x12_Pin, Connector_PinHeader_2.54mm:PinHeader_1x12_P2.54mm_Vertical, symbol Connector:Conn_01x12_Pin
- added J1: Header1, Connector_PinHeader_2.54mm:PinHeader_1x13_P2.54mm_Vertical, symbol Connector:Conn_01x13_Pin
- added J2: Header2, Connector_PinHeader_2.54mm:PinHeader_1x13_P2.54mm_Vertical, symbol Connector:Conn_01x13_Pin
- LED2: renamed from LED1; value PWR -> USR
- renumbered C7 to C1, C8 to C2, C1 to C3, C2 to C4, C3 to C5, C4 to C6, C5 to C7, C6 to C8, J1 to J3, LED to LED1, R3 to R1, R1 to R2, R2 to R3, R5 to R4, R6 to R5, R4 to R6, SW2 to SW1, SW1 to SW2, U2 to U1, U1 to U2, J2 to USB1
Connections:
- net +3.3V: now also J1.2 (Pin_2), J2.9 (Pin_9)
- net BOOT0 BTN: now also J1.4 (Pin_4)
- net GND: now also J1.1 (Pin_1), J1.3 (Pin_3), J1.8 (Pin_8), J2.2 (Pin_2), J2.3 (Pin_3), J2.8 (Pin_8)
- net OSC_IN: now also J1.5 (Pin_5)
- net OSC_OUT: now also J1.6 (Pin_6)
- net PA0: now also J1.9 (Pin_9)
- net PA1: now also J1.10 (Pin_10)
- net PA11: now also J2.7 (Pin_7)
- net PA12: now also J2.6 (Pin_6)
- net PA2: now also J1.11 (Pin_11)
- net PA3: now also J1.12 (Pin_12)
- net PA4: now also J1.13 (Pin_13)
- net PA5: now also J2.13 (Pin_13)
- net PA6: now also J2.12 (Pin_12)
- net PA7: now also J2.11 (Pin_11)
- net Reset BTN: now also J1.7 (Pin_7)
- net SWCLK: now also J2.4 (Pin_4)
- net SWDIO: now also J2.5 (Pin_5)
- net USR_LED: now also J2.10 (Pin_10)
- net VBUS: now also J2.1 (Pin_1)

Commit message: board ready
Parts:
- USB1: footprint Connector_USB:USB_C_Receptacle_Palconn_UTC16-G -> Connector_USB:USB_C_Receptacle_HCTL_HC-TYPE-C-16P-01A
- Y1: footprint Crystal:Crystal_SMD_5032-2Pin_5.0x3.2mm_HandSoldering -> Crystal:Crystal_SMD_5032-2Pin_5.0x3.2mm
Changed lines of the file:
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@@
 			)
 		)
-		(property "Footprint" "Connector_USB:USB_C_Receptacle_Palconn_UTC16-G"
+		(property "Footprint" "Connector_USB:USB_C_Receptacle_HCTL_HC-TYPE-C-16P-01A"
 			(at 214.63 125.73 0)
 			(effects
@@
 			)
 		)
-		(property "Footprint" "Crystal:Crystal_SMD_5032-2Pin_5.0x3.2mm_HandSoldering"
+		(property "Footprint" "Crystal:Crystal_SMD_5032-2Pin_5.0x3.2mm"
 			(at 48.26 91.44 0)
 			(effects
